Commit message: Update description

File: baxter_description/urdf/pedestal/pedestal.xacro (robot description, xacro)
@@ -30,11 +30,3 @@
     <child link="pedestal"/>
   </joint>
-  <xacro:if value="$(arg gazebo)">
-    <!-- When using the pedistal, fix Baxter to Gazebo world with 'base' frame -->
-    <link name="world"/>
-    <joint name="fixed" type="fixed">
-      <parent link="world"/>
-      <child link="base"/>
-    </joint>
-  </xacro:if>
 </robot>
